Commit message: Implementation of dynamic model and controller

File: uuv_simulation/models/uuv_gamma.urdf (robot description, URDF)
Before this commit: robot boat, 1 links, 0 joints
Links:
- link uuv: geometry visual mesh filename=package://uuv_simulation/models/meshes/VTEC_U-II_GAMMA.STL scale=0.001 0.001 0.001
