Commit message: 6DOF uuv class works correctly. 6DOF PID Controller works correctly, but better gains may be required (or there could be a bug somewhere). Tested for setpoint regulation. ASMC still requires implementation. Trajectory tracking case will be developed soon

File: models/vtec_u3.urdf (robot description, URDF)
Before this commit: robot uuv, 1 links, 0 joints
Links:
- link uuv: geometry visual mesh filename=package://vanttec_uuv/models/meshes/VTEC_U-II_GAMMA.STL scale=0.001 0.001 0.001
