Commit message: changes

File: models/uuv_gamma.urdf (robot description, URDF)
Before this commit: robot uuv, 1 links, 0 joints
Links:
- link uuv: geometry visual mesh filename=package://vanttec_uuv/models/meshes/VTEC_U-II_.STL scale=0.001 0.001 0.001

Commit message: integration update

File: models/uuv_gamma.urdf (robot description, URDF)
Before this commit: robot uuv, 1 links, 0 joints
Links:
- removed link uuv
- added link vtec_u3_base_link; visual mesh filename=package://vanttec_uuv/models/meshes/VTEC_U-II_GAMMA.STL scale=0.001 0.001 0.001
