Commit message: vanttec_controllers successfully integrated in uuv_control

File: uuv_control/models/vtec_u3.urdf (robot description, URDF)
Before this commit: robot uuv, 1 links, 0 joints
Links:
- link uuv: geometry visual mesh filename=package://uuv_control/models/meshes/VTEC_U-II_GAMMA.STL scale=0.001 0.001 0.001
