Commit message: Simualted environments are now working

File: uuv_gazebo/urdf/bin1.xacro (robot description, xacro)
@@ -3,5 +3,5 @@
 <!--Change .dae to binopen.dae, bintapadod.dae, bintapadoi.dae depending on the situation-->
 <!-- Introducir meshes -->
-<xacro:property name="visual_mesh_file" value="file://$(find uv_worlds)/models/props//bintapadoi.dae" />
+<xacro:property name="visual_mesh_file" value="file://$(find uuv_gazebo)/models/props//bintapadoi.dae" />
 <!-- <origin xyz="0.085 (0 -0.085) 0 0" rpy="0.0 0.0 1.57075"/> -->
 <link name="bin1_base">

File: uuv_gazebo/urdf/bin2.xacro (robot description, xacro)
@@ -2,5 +2,5 @@
 <robot name="bin_2" xmlns:xacro="http://www.ros.org/wiki/xacro">
 <!-- Introducir meshes -->
-<xacro:property name="visual_mesh_file" value="file://$(find uv_worlds)/models/props//bin02.dae" />
+<xacro:property name="visual_mesh_file" value="file://$(find uuv_gazebo)/models/props//bin02.dae" />
 <!-- <origin xyz="0.085 (0 -0.085) 0 0" rpy="0.0 0.0 1.57075"/> -->
 <link name="bin2_base">

File: uuv_gazebo/urdf/bottle.xacro (robot description, xacro)
@@ -2,5 +2,5 @@
 <robot name="bottle" xmlns:xacro="http://www.ros.org/wiki/xacro">
 <!-- Introducir meshes -->
-<xacro:property name="visual_mesh_file" value="file://$(find uv_worlds)/models/props/bottle/water_bottle.dae" />
+<xacro:property name="visual_mesh_file" value="file://$(find uuv_gazebo)/models/props/bottle/water_bottle.dae" />
 <!-- <origin xyz="0.085 (0 -0.085) 0 0" rpy="0.0 0.0 1.57075"/> -->
 <link name="bottle_base">

File: uuv_gazebo/urdf/buoy.xacro (robot description, xacro)
@@ -2,5 +2,5 @@
 <robot name="buoy_1" xmlns:xacro="http://www.ros.org/wiki/xacro">
 <!-- Introducir meshes -->
-<xacro:property name="visual_mesh_file" value="file://$(find uv_worlds)/models/props//buoy1.dae" />
+<xacro:property name="visual_mesh_file" value="file://$(find uuv_gazebo)/models/props//buoy1.dae" />
 <!-- <origin xyz="0.085 (0 -0.085) 0 0" rpy="0.0 0.0 1.57075"/> -->
 <link name="buoy1_base">

File: uuv_gazebo/urdf/buoy2.xacro (robot description, xacro)
@@ -2,5 +2,5 @@
 <robot name="buoy_2" xmlns:xacro="http://www.ros.org/wiki/xacro">
 <!-- Introducir meshes -->
-<xacro:property name="visual_mesh_file" value="file://$(find uv_worlds)/models/props//buoy2.dae" />
+<xacro:property name="visual_mesh_file" value="file://$(find uuv_gazebo)/models/props//buoy2.dae" />
 <!-- <origin xyz="0.085 (0 -0.085) 0 0" rpy="0.0 0.0 1.57075"/> -->
 <link name="buoy2_base">

File: uuv_gazebo/urdf/gate.xacro (robot description, xacro)
@@ -2,5 +2,5 @@
 <robot name="gate_1" xmlns:xacro="http://www.ros.org/wiki/xacro">
 <!-- Introducir meshes -->
-<xacro:property name="visual_mesh_file" value="file://$(find uv_worlds)/models/gate1/mygate1.dae" />
+<xacro:property name="visual_mesh_file" value="file://$(find uuv_gazebo)/models/gate1/mygate1.dae" />
 <!-- <origin xyz="0.085 (0 -0.085) 0 0" rpy="0.0 0.0 1.57075"/> -->
 <link name="gate_base">

File: uuv_gazebo/urdf/gman.xacro (robot description, xacro)
@@ -1,5 +1,5 @@
 <?xml version="1.0"?>
 <robot name="gman_target" xmlns:xacro="http://www.ros.org/wiki/xacro">
-    <xacro:property name="visual_mesh_file" value="file://$(find props_gazebo)/meshes/gman.dae" />
+    <xacro:property name="visual_mesh_file" value="file://$(find uuv_gazebo)/meshes/gman.dae" />
     <!-- <xacro:property name="collision_mesh_file" value="file://$(find props_gazebo)/meshes/gman.dae"/> -->
     <link name="base_link">

File: uuv_gazebo/urdf/octagon.xacro (robot description, xacro)
@@ -2,5 +2,5 @@
 <robot name="octagon_1" xmlns:xacro="http://www.ros.org/wiki/xacro">
 <!-- Introducir meshes -->
-<xacro:property name="visual_mesh_file" value="file://$(find uv_worlds)/models/props//Myoctagon2.dae" />
+<xacro:property name="visual_mesh_file" value="file://$(find uuv_gazebo)/models/props/Myoctagon2.dae" />
 <!-- <origin xyz="0.085 (0 -0.085) 0 0" rpy="0.0 0.0 1.57075"/> -->
 <link name="octagon_base">

File: uuv_gazebo/urdf/torpedos1.xacro (robot description, xacro)
@@ -2,5 +2,5 @@
 <robot name="torpedos_1" xmlns:xacro="http://www.ros.org/wiki/xacro">
 <!-- Introducir meshes -->
-<xacro:property name="visual_mesh_file" value="file://$(find uv_worlds)/models/props//finaltorpedos.dae" />
+<xacro:property name="visual_mesh_file" value="file://$(find uuv_gazebo)/models/props/finaltorpedos.dae" />
 <!-- <origin xyz="0.085 (0 -0.085) 0 0" rpy="0.0 0.0 1.57075"/> -->
 <link name="torpedos1_base">

File: uuv_gazebo/urdf/torpedos2.xacro (robot description, xacro)
@@ -2,5 +2,5 @@
 <robot name="torpedos_2" xmlns:xacro="http://www.ros.org/wiki/xacro">
 <!-- Introducir meshes -->
-<xacro:property name="visual_mesh_file" value="file://$(find uv_worlds)/models/props//Mytorpedos2.dae" />
+<xacro:property name="visual_mesh_file" value="file://$(find uuv_gazebo)/models/props/Mytorpedos2.dae" />
 <!-- <origin xyz="0.085 (0 -0.085) 0 0" rpy="0.0 0.0 1.57075"/> -->
 <link name="torpedos2_base">
