Commit message: More changes

File: uuv_description/robots/vtec_u3.xacro (robot description, xacro)
@@ -4,6 +4,6 @@
   <xacro:arg name="namespace" default="vtec_u3"/>
   <xacro:arg name="inertial_reference_frame" default="world_ned"/>
-  <xacro:include filename="$(find vehicle_descriptions)/urdf/UUVs/vtec_u3_base.xacro"/>
-  <xacro:include filename="$(find vehicle_descriptions)/urdf/UUVs/vtec_u3_sensors.xacro"/>
+  <xacro:include filename="$(find uuv_description)/urdf/UUVs/vtec_u3_base.xacro"/>
+  <xacro:include filename="$(find uuv_description)/urdf/UUVs/vtec_u3_sensors.xacro"/>
   <virtual_joint name="world_joint" type="planar" parent_frame="world_ned" child_link="vtec_u3_base_link"/>
   <xacro:vtec_u3_base namespace="$(arg namespace)"/>

File: uuv_description/urdf/UUVs/vtec_u3_base.xacro (robot description, xacro)
@@ -11,5 +11,5 @@
     the mesh pose will have to be corrected below in the <visual> block.
   -->
-  <xacro:property name="visual_mesh_file" value="file://$(find vehicle_descriptions)/meshes/vtec_u3.dae"/>
+  <xacro:property name="visual_mesh_file" value="file://$(find uuv_description)/meshes/vtec_u3.dae"/>
   <!--
     Collision geometry mesh, usually in STL format (it is recommended to keep
@@ -17,5 +17,5 @@
     regarding the computation of collision forces)
   -->
-  <xacro:property name="collision_mesh_file" value="file://$(find vehicle_descriptions)/meshes/vtec_u3.stl"/>
+  <xacro:property name="collision_mesh_file" value="file://$(find uuv_description)/meshes/vtec_u3.stl"/>
   <xacro:macro name="vtec_u3_base" params="namespace">
       <link name="${namespace}_base_link">

File: uuv_description/urdf/UUVs/vtec_u3_sensors.xacro (robot description, xacro)
@@ -1,5 +1,5 @@
 <?xml version="1.0"?>
 <robot xmlns:xacro="http://www.ros.org/wiki/xacro">
-  <xacro:include filename="$(find uuv_sensor_ros_plugins)/urdf/sensor_snippets.xacro"/>
+  <xacro:include filename="$(find uuv_gazebo)/plugins/uuv_sensor_plugins/uuv_sensor_ros_plugins/urdf/sensor_snippets.xacro"/>
   <!-- Sensor macros in the package uuv_sensor_ros_plugins/urdf -->
   <xacro:macro name="vtec_u3_sensors" params="namespace">

File: uuv_description/urdf/UUVs/vtec_u3_shooter.xacro (robot description, xacro)
@@ -2,5 +2,5 @@
 <robot xmlns:xacro="http://www.ros.org/wiki/xacro">
   <xacro:macro name="vtec_u3_shooter" params="parent">
-    <xacro:property name="visual_mesh_file" value="file://$(find vehicle_descriptions)/meshes/shooter/shooter_base.dae" />
+    <xacro:property name="visual_mesh_file" value="file://$(find uuv_description)/meshes/shooter/shooter_base.dae" />
     <!-- <xacro:property name="collision_mesh_file" value="file://$(find vehicle_descriptions)/meshes/shooter/shooter_base.dae"/> -->
     <gazebo reference="shooter_base_link">
