Commit message: Working version of Gazebo with UUV and the realsense_gazebo_plugin

File: uuv_description/urdf/UUVs/vtec_u3_base.xacro (robot description, xacro)
@@ -35,5 +35,5 @@
           <origin xyz="${geocenter}" rpy="0 0 0"/>
           <geometry>
-            <mesh filename="${visual_mesh_file}" scale="0.001 0.001 0.001" />
+            <mesh filename="${visual_mesh_file}" scale="1 1 1" />
           </geometry>
         </visual>

File: uuv_description/urdf/UUVs/vtec_u3_sensors.xacro (robot description, xacro)
@@ -7,9 +7,8 @@
     <xacro:name_sensor ... > name_sensor found on the urdf/sensor_snippets.xacro.
     -->
-    <!-- Realsense R200 Camera
+    <!-- Realsense R200 Camera -->
     <xacro:realsense_camera namespace="${namespace}" parent_link="${namespace}_base_link" suffix="front">
-      <origin xyz="0.19281 0.01961 0.06659" rpy="0 0 0"/>
+      <origin xyz="0 0 0.18" rpy="0 0 1.57"/>
     </xacro:realsense_camera>
--->
   </xacro:macro>
 </robot>

File: uuv_gazebo/plugins/realsense_gazebo_plugin/urdf/multi_rs200_simulation.xacro (robot description, xacro)
@@ -3,5 +3,5 @@
     <link name="world"/>
     <!-- Import macro for realsense-RS200 camera-->
-    <xacro:include filename="$(find realsense_gazebo_plugin)/urdf/realsense-RS200.macro.xacro"/>
+    <xacro:include filename="$(find uuv_gazebo)/plugins/realsense_gazebo_plugin/urdf/realsense-RS200.macro.xacro"/>
     <!-- Create two camera instances -->
     <xacro:realsense-rs200 prefix="left_" parent="world">

File: uuv_gazebo/plugins/realsense_gazebo_plugin/urdf/rs200_simulation.xacro (robot description, xacro)
@@ -7,5 +7,5 @@
     <link name="world"/>
     <!-- Import macro for realsense-RS200 camera-->
-    <xacro:include filename="$(find realsense_gazebo_plugin)/urdf/realsense-RS200.macro.xacro"/>
+    <xacro:include filename="$(find uuv_gazebo)/plugins/realsense_gazebo_plugin/urdf/realsense-RS200.macro.xacro"/>
     <!-- Create camera instance -->
     <xacro:realsense-rs200 prefix="" parent="world">

File: uuv_gazebo/plugins/uuv_sensor_plugins/uuv_sensor_ros_plugins/urdf/camera_snippets.xacro (robot description, xacro)
@@ -53,5 +53,5 @@
       scale="1.0">
       <inertia ixx="0.00001" ixy="0.0" ixz="0.0" iyy="0.00001" iyz="0.0" izz="0.00001" />
-      <xacro:insert_block name="origin" />>
+      <xacro:insert_block name="origin" />
     </xacro:regular_camera_plugin_macro>
   </xacro:macro>
@@ -69,5 +69,5 @@
       <visual>
         <geometry>
-          <mesh filename="file://$(find uuv_sensor_ros_plugins)/meshes/oe14-372.dae" scale="${scale} ${scale} ${scale}"/>
+          <mesh filename="file://$(find uuv_gazebo)/plugins/uuv_sensor_plugins/uuv_sensor_ros_plugins/meshes/oe14-372.dae" scale="${scale} ${scale} ${scale}"/>
         </geometry>
       </visual>
@@ -154,5 +154,5 @@
       <visual>
         <geometry>
-          <mesh filename="file://$(find uuv_sensor_ros_plugins)/meshes/oe14-372.dae" scale="1 1 1"/>
+          <mesh filename="file://$(find uuv_gazebo)/plugins/uuv_sensor_plugins/uuv_sensor_ros_plugins/meshes/oe14-372.dae" scale="1 1 1"/>
         </geometry>
       </visual>

File: uuv_gazebo/plugins/uuv_sensor_plugins/uuv_sensor_ros_plugins/urdf/realsense_camera.xacro (robot description, xacro)
@@ -50,5 +50,5 @@
             <origin rpy="0 0 0" xyz="0 0 0"/>
             <geometry>
-                <mesh filename="package://realsense_gazebo_plugin/models/realsense_camera/meshes/realsense.dae"/>
+                <mesh filename="package://uuv_gazebo/plugins/realsense_gazebo_plugin/models/realsense_camera/meshes/realsense.dae"/>
             </geometry>
         </visual>
