Commit message: Changes before merging

File: uuv_description/urdf/UUVs/vtec_u3_sensors.xacro (robot description, xacro)
@@ -11,4 +11,7 @@
       <origin xyz="0 0 0.18" rpy="0 0 1.57"/>
     </xacro:realsense_camera>
+    <xacro:default_pressure_macro namespace="${namespace}" parent_link="${namespace}_base_link">
+      <origin xyz="0 0 0" rpy="0 0 1.57"/>
+    </xacro:default_pressure_macro>
   </xacro:macro>
 </robot>

File: uuv_gazebo/plugins/uuv_sensor_plugins/uuv_sensor_ros_plugins/urdf/pressure_snippets.xacro (robot description, xacro)
@@ -36,5 +36,5 @@
       kPaPerM="9.80638">
       <inertia ixx="0.00001" ixy="0.0" ixz="0.0" iyy="0.00001" iyz="0.0" izz="0.00001" />
-      <xacro:insert_block name="origin" />>
+      <xacro:insert_block name="origin" />
     </xacro:pressure_plugin_macro>
   </xacro:macro>
@@ -69,18 +69,14 @@
       <visual>
         <geometry>
-          <mesh filename="file://$(find uuv_sensor_ros_plugins)/meshes/pressure.dae" scale="0.1 0.1 0.1"/>
+          <mesh filename="file://$(find uuv_gazebo)/plugins/uuv_sensor_plugins/uuv_sensor_ros_plugins/meshes/pressure.dae" scale="0.1 0.1 0.1"/>
         </geometry>
       </visual>
       <xacro:no_collision/>
     </link>
-    <gazebo reference="${namespace}/pressure${suffix}_link">>
+    <gazebo reference="${namespace}/pressure${suffix}_link">
       <turnGravityOff>1</turnGravityOff>
     </gazebo>
     <joint name="${namespace}/pressure${suffix}_joint" type="revolute">
       <xacro:insert_block name="origin" />
-      <parent link="${parent_link}" />
-      <child link="${namespace}/pressure${suffix}_link" />
-      <limit upper="0" lower="0" effort="0" velocity="0" />
-      <axis xyz="1 0 0"/>
     </joint>
     <gazebo>

Commit message: Major changes and a working implementation of the pose_3d_plugin

File: uuv_description/urdf/UUVs/vtec_u3_sensors.xacro (robot description, xacro)
@@ -11,7 +11,14 @@
       <origin xyz="0 0 0.18" rpy="0 0 1.57"/>
     </xacro:realsense_camera>
-    <!--xacro:default_pressure_macro namespace="${namespace}" parent_link="${namespace}_base_link">
-      <origin xyz="0 0 0" rpy="0 0 1.57"/>
-    </xacro:default_pressure_macro> -->
+    <gazebo>
+      <plugin name="pose_3d_plugin" filename="libgazebo_ros_p3d.so">
+      <robotNamespace>${namespace}</robotNamespace>
+      <bodyName>${namespace}_base_link</bodyName>
+      <topicName>pose_gt</topicName>
+      <frameName>world</frameName>
+      <gaussianNoise>0.0</gaussianNoise>
+      <updateRate>30</updateRate>
+      </plugin>
+    </gazebo>
   </xacro:macro>
 </robot>

File: uuv_gazebo/plugins/uuv_sensor_plugins/uuv_sensor_ros_plugins/urdf/imu_snippets.xacro (robot description, xacro)
@@ -84,5 +84,5 @@
       update_rate="50">
       <inertia ixx="0.00001" ixy="0.0" ixz="0.0" iyy="0.00001" iyz="0.0" izz="0.00001" />
-      <xacro:insert_block name="origin" />>
+      <xacro:insert_block name="origin" />
     </xacro:imu_plugin_macro>
   </xacro:macro>

File: uuv_gazebo/plugins/uuv_sensor_plugins/uuv_sensor_ros_plugins/urdf/pressure_snippets.xacro (robot description, xacro)
@@ -78,5 +78,9 @@
     </gazebo>
     <joint name="${namespace}/pressure${suffix}_joint" type="revolute">
-      <xacro:insert_block name="origin" />
+      <xacro:insert_block name="origin"/>
+      <parent link="${parent_link}"/>
+      <child link="${namespace}/pressure${suffix}_link"/>
+      <limit upper="0" lower="0" effort="0" velocity="0" />
+      <axis xyz="1 0 0"/>
     </joint>
     <gazebo>
